Commit message: baseline before simulation performance optimization

File: src/humbleble_ws/amir740_ros/amir_description/urdf/amir_for_rover.xacro (robot description, xacro)
@@ -522,7 +522,12 @@
 </joint> -->
 <!-- end of outer joint -->
-<!-- D435 depth camera mounted at end effector (tcp_link) -->
-<xacro:sensor_d435 parent="tcp_link" name="d435" topics_ns="d435" use_nominal_extrinsics="true">
-  <origin xyz="0 -0.06 0.03" rpy="0 0 1.5708"/>
-</xacro:sensor_d435>
+<!-- D435 depth camera mounted at end effector (tcp_link).  The cooperative
+     transport simulation does not consume camera data, so it can be omitted
+     to avoid rendering 1280x720 RGB-D images for both robots. -->
+<xacro:arg name="enable_d435" default="true"/>
+<xacro:if value="$(arg enable_d435)">
+  <xacro:sensor_d435 parent="tcp_link" name="d435" topics_ns="d435" use_nominal_extrinsics="true">
+    <origin xyz="0 -0.06 0.03" rpy="0 0 1.5708"/>
+  </xacro:sensor_d435>
+</xacro:if>
 </robot>

File: src/humbleble_ws/amir740_ros/amir_description/urdf/amir_mecanum3_sim.xacro (robot description, xacro)
@@ -6,4 +6,5 @@
        TF frame ID は共通名のまま、launch 側でTF topicをnamespace分離する。 -->
   <xacro:arg name="namespace" default=""/>
+  <xacro:arg name="enable_wrist_ft" default="true"/>
   <!-- メカナムローバー URDF
        mecanum3.gazebo (gz_ros2_control-system) と
@@ -44,4 +45,5 @@
       </command_interface>
       <state_interface name="position">
+        <!-- Common AMIR spawn posture (radians): Q_HOME[0]. -->
         <param name="initial_value">0.0</param>
       </state_interface>
@@ -54,5 +56,6 @@
       </command_interface>
       <state_interface name="position">
-        <param name="initial_value">0.0</param>
+        <!-- Common AMIR spawn posture (radians): Q_HOME[1]. -->
+        <param name="initial_value">1.4</param>
       </state_interface>
       <state_interface name="velocity"/>
@@ -64,5 +67,6 @@
       </command_interface>
       <state_interface name="position">
-        <param name="initial_value">0.0</param>
+        <!-- Common AMIR spawn posture (radians): Q_HOME[2]. -->
+        <param name="initial_value">-1.6</param>
       </state_interface>
       <state_interface name="velocity"/>
@@ -74,5 +78,6 @@
       </command_interface>
       <state_interface name="position">
-        <param name="initial_value">0.0</param>
+        <!-- Common AMIR spawn posture (radians): Q_HOME[3]. -->
+        <param name="initial_value">0.2</param>
       </state_interface>
       <state_interface name="velocity"/>
@@ -84,5 +89,6 @@
       </command_interface>
       <state_interface name="position">
-        <param name="initial_value">0.0</param>
+        <!-- Common AMIR spawn posture (radians): Q_HOME[4]. -->
+        <param name="initial_value">1.570796</param>
       </state_interface>
       <state_interface name="velocity"/>
@@ -160,4 +166,5 @@
   <!-- Joint_5 is the wrist joint directly upstream of the gripper.  Gazebo
        publishes its transmitted six-axis wrench in the gripper frame. -->
+  <xacro:if value="$(arg enable_wrist_ft)">
   <gazebo reference="Joint_5">
     <sensor name="wrist_ft_sensor" type="force_torque">
@@ -171,4 +178,5 @@
     </sensor>
   </gazebo>
+  </xacro:if>
   <!-- Gazebo Fortress's contact message identifies the colliding bodies but
        does not expose the solver wrench.  These joint sensors provide the

Commit message: Evaluate gripper collision simplification and retain nine-box baseline

File: src/humbleble_ws/amir740_ros/amir_description/urdf/amir_for_rover.xacro (robot description, xacro)
@@ -7,4 +7,6 @@
 <!-- <xacro:include filename="$(find amir_description)/urdf/amir_mecanum3.gazebo.xacro" />
 <xacro:include filename="$(find amir_description)/urdf/amir_mecanum3.gazebo_ros2_control.xacro" /> -->
+<xacro:arg name="finger_collision_boxes" default="9"/>
+<xacro:property name="finger_collision_boxes" value="$(arg finger_collision_boxes)"/>
 <!-- Emit one identical visual/collision pair.  A stack of these boxes follows
      the original STL finger silhouette while retaining stable primitive
@@ -18,4 +20,5 @@
     <material name="silver-amir"/>
   </visual>
+  <xacro:if value="${int(finger_collision_boxes) == 9}">
   <collision>
     <origin xyz="${xyz}" rpy="0 0 0"/>
@@ -23,4 +26,10 @@
       <box size="${size}"/>
     </geometry>
+  </collision>
+  </xacro:if>
+</xacro:macro>
+<xacro:macro name="finger_collision_box" params="xyz size">
+  <collision><origin xyz="${xyz}" rpy="0 0 0"/>
+    <geometry><box size="${size}"/></geometry>
   </collision>
 </xacro:macro>
@@ -299,4 +308,13 @@
   <xacro:finger_box xyz="-0.025967 0.045477 0.000403"
                     size="0.003800 0.006000 0.050000"/>
+  <!-- Collision experiment: original contact pad retained exactly in 3-box mode. -->
+  <xacro:if value="${int(finger_collision_boxes) == 3}">
+    <xacro:finger_collision_box xyz="-0.018767 0.022477 0.000403" size="0.018200 0.008000 0.050000"/>
+    <xacro:finger_collision_box xyz="-0.011617 -0.001023 0.000403" size="0.032500 0.039000 0.050000"/>
+    <xacro:finger_collision_box xyz="-0.021067 0.037477 0.000403" size="0.013600 0.022000 0.050000"/>
+  </xacro:if>
+  <xacro:if value="${int(finger_collision_boxes) == 1}">
+    <xacro:finger_collision_box xyz="-0.011617 0.013977 0.000403" size="0.032500 0.069000 0.050000"/>
+  </xacro:if>
 </link>
 <link name="finger_left_1">
@@ -330,4 +348,13 @@
   <xacro:finger_box xyz="0.025600 0.045000 0.000403"
                     size="0.003800 0.006000 0.050000"/>
+  <!-- Collision experiment: original contact pad retained exactly in 3-box mode. -->
+  <xacro:if value="${int(finger_collision_boxes) == 3}">
+    <xacro:finger_collision_box xyz="0.018400 0.022000 0.000403" size="0.018200 0.008000 0.050000"/>
+    <xacro:finger_collision_box xyz="0.011250 -0.001500 0.000403" size="0.032500 0.039000 0.050000"/>
+    <xacro:finger_collision_box xyz="0.020700 0.037000 0.000403" size="0.013600 0.022000 0.050000"/>
+  </xacro:if>
+  <xacro:if value="${int(finger_collision_boxes) == 1}">
+    <xacro:finger_collision_box xyz="0.011250 0.013500 0.000403" size="0.032500 0.069000 0.050000"/>
+  </xacro:if>
 </link>
 <!-- end of inner link -->

File: src/humbleble_ws/amir740_ros/amir_description/urdf/amir_mecanum3_sim.xacro (robot description, xacro)
@@ -248,12 +248,28 @@
       </contact>
     </sensor>
+    <xacro:if value="${int(finger_collision_boxes) > 1}">
     <xacro:finger_segment_contact side="left" suffix="_1" collision_suffix="_1"/>
+    </xacro:if>
+    <xacro:if value="${int(finger_collision_boxes) > 2}">
     <xacro:finger_segment_contact side="left" suffix="_2" collision_suffix="_2"/>
+    </xacro:if>
+    <xacro:if value="${int(finger_collision_boxes) > 3}">
     <xacro:finger_segment_contact side="left" suffix="_3" collision_suffix="_3"/>
+    </xacro:if>
+    <xacro:if value="${int(finger_collision_boxes) > 4}">
     <xacro:finger_segment_contact side="left" suffix="_4" collision_suffix="_4"/>
+    </xacro:if>
+    <xacro:if value="${int(finger_collision_boxes) > 5}">
     <xacro:finger_segment_contact side="left" suffix="_5" collision_suffix="_5"/>
+    </xacro:if>
+    <xacro:if value="${int(finger_collision_boxes) > 6}">
     <xacro:finger_segment_contact side="left" suffix="_6" collision_suffix="_6"/>
+    </xacro:if>
+    <xacro:if value="${int(finger_collision_boxes) > 7}">
     <xacro:finger_segment_contact side="left" suffix="_7" collision_suffix="_7"/>
+    </xacro:if>
+    <xacro:if value="${int(finger_collision_boxes) > 8}">
     <xacro:finger_segment_contact side="left" suffix="_8" collision_suffix="_8"/>
+    </xacro:if>
   </gazebo>
   <gazebo reference="finger_right_1">
@@ -284,12 +300,28 @@
       </contact>
     </sensor>
+    <xacro:if value="${int(finger_collision_boxes) > 1}">
     <xacro:finger_segment_contact side="right" suffix="_1" collision_suffix="_1"/>
+    </xacro:if>
+    <xacro:if value="${int(finger_collision_boxes) > 2}">
     <xacro:finger_segment_contact side="right" suffix="_2" collision_suffix="_2"/>
+    </xacro:if>
+    <xacro:if value="${int(finger_collision_boxes) > 3}">
     <xacro:finger_segment_contact side="right" suffix="_3" collision_suffix="_3"/>
+    </xacro:if>
+    <xacro:if value="${int(finger_collision_boxes) > 4}">
     <xacro:finger_segment_contact side="right" suffix="_4" collision_suffix="_4"/>
+    </xacro:if>
+    <xacro:if value="${int(finger_collision_boxes) > 5}">
     <xacro:finger_segment_contact side="right" suffix="_5" collision_suffix="_5"/>
+    </xacro:if>
+    <xacro:if value="${int(finger_collision_boxes) > 6}">
     <xacro:finger_segment_contact side="right" suffix="_6" collision_suffix="_6"/>
+    </xacro:if>
+    <xacro:if value="${int(finger_collision_boxes) > 7}">
     <xacro:finger_segment_contact side="right" suffix="_7" collision_suffix="_7"/>
+    </xacro:if>
+    <xacro:if value="${int(finger_collision_boxes) > 8}">
     <xacro:finger_segment_contact side="right" suffix="_8" collision_suffix="_8"/>
+    </xacro:if>
   </gazebo>
 </robot>
